File: eduBoard.sch (EAGLE design)
At the start: 63 parts, among them IC1 NCP1117ST50T3G, IC3 ATMEGA2560-16AU, IC4 ATMEGA16U2-MU, IC6 LP2985-33DBVR, IC7 LMV358IDGKR, T1 FDN340P, X1 POWERSUPPLY_DC21MMX, X2 USB-B_TH, Y1 CSTCE16M0V53-R0 16MHZ, Y2 16MHz

Commit message: nicer mega shield
Parts:
- removed C1, C14, C15: 22p, SmartPrj:C-EU0603-RND
- removed C10, C13: 1u, SmartPrj:C-EU0603-RND
- removed C11, C12, C2, C3, C4, C5, C6, C7, C8, C9: 100n, SmartPrj:C-EU0603-RND
- removed D1: M7, diode:DIODE-SMB
- removed D2, D3: CD1206-S01575, diode:DIODE-MINIMELF
- removed F1: MF-MSMF050-2 500mA, rcl:L-EUL1812
- removed GROUND, RESET-EN: (no value), jumper:SJ
- removed IC1: NCP1117ST50T3G, linear:MC33269ST-3.3T3
- removed IC3: ATMEGA2560-16AU, SmartPrj:ATMEGA25602560-16AU
- removed IC4: ATMEGA16U2-MU, SmartPrj:ATMEGA16U2-MU
- removed IC6: LP2985-33DBVR, SmartPrj:LP2985-XXDBVR33
- removed IC7: LMV358IDGKR, linear:LMV358MMX
- removed L, RX, TX: YELLOW, led:LEDCHIP-LED0805
- removed L1: BLM21, wuerth-elektronik:WE-CBF_0805
- removed ON: GREEN, led:LEDCHIP-LED0805
- removed PC1, PC2: 47u, rcl:CPOL-EUD
- removed R1, R2: 1M, SmartPrj:R-EU_R0603
- removed RESET: TS42031-160R-TR-7260, SmartPrj:TS42
- removed RN1, RN5: 10K, resistor-dil:4R-NCAT16
- removed RN2: 22R, resistor-dil:4R-NCAY16
- removed RN3, RN4: 1k, resistor-dil:4R-NCAY16
- removed T1: FDN340P, zetex:PMOSSOT23
- removed U$1: DISCLAIMER, SmartPrj:DISCLAIMER
- removed X1: POWERSUPPLY_DC21MMX, SmartPrj:POWERSUPPLY_DC21MMX
- removed X2: USB-B_TH, SmartPrj:PN61729
- removed Y1: CSTCE16M0V53-R0 16MHZ, SmartPrj:RESONATORMU
- removed Y2: 16MHz, SmartPrj:XTAL/S
- removed Z1, Z2: CG0603MLC-05E, varistor:VARISTORCN0603
Connections:
- removed net CMP: C12.2, IC7B.+IN, RN5C.1, RN5D.2
- removed net D+: RN2D.2, X2.3, Z2.2
- removed net D-: RN2A.2, X2.2, Z1.2
- removed net DTR: C7.1, IC4.(CTS/HWB/AIN6/TO/INT7)PD7, RN3D.1
- removed net GATE_CMD: IC7B.OUT, T1.G
- removed net L13: IC7A.-IN, IC7A.OUT, RN3B.2
- removed net M8RXD: IC4.(TXD1/INT3)PD3, RN4B.2
- removed net M8TXD: IC4.(RXD1/AIN1/INT2)PD2, RN4A.2
- removed net N$2: L.A, RN3B.1
- removed net N$54: RN4D.1, RX.A
- removed net N$55: RN4C.1, TX.A
- removed net PWRIN: D1.A, X1.2
- removed net RD+: IC4.D+, RN2D.1
- removed net RD-: IC4.D-, RN2A.1
- removed net RXL: IC4.(INT5/AIN3)PD4, RX.C
- removed net TXL: IC4.(XCK/AIN4/PCINT12)PD5, TX.C
- removed net UGND: C10.2, GROUND.1, IC4.UGND, L1.1, X2.4
- removed net USBVCC: C8.1, F1.1, IC4.UVCC, T1.D
- removed net USHIELD: L1.2, X2.P$1, X2.P$2, Z1.1, Z2.1
- removed net VUCAP: C10.1, IC4.UCAP
- removed net XT1: C14.1, IC4.XTAL1, R2.1, Y2.2
- removed net XT2: C15.1, IC4.XTAL2(PC0), R2.2, Y2.1
- removed net XTAL1: IC3.XTAL1, R1.1, Y1.3
- removed net XTAL2: IC3.XTAL2, R1.2, Y1.1
- removed net XVCC: F1.2, X2.1
- net +3V3: no longer C13.2, IC6.OUT, IC7B.-IN
- net +5V: no longer C11.2, C4.1, C5.1, C6.1, C9.1, D2.C, D3.C, IC1.OUT, IC1.OUT@1, IC3.AVCC, IC3.VCC, IC3.VCC1, IC3.VCC2, IC3.VCC3, IC4.AVCC, IC4.VCC, IC6.IN, IC6.ON/!OFF, IC7P.V+, PC2.+, RN1B.2, RN1C.2, RN3A.1, RN4C.2, RN4D.2, RN5A.2, RN5B.1, T1.S
- net 8PB4: no longer IC4.(T1/PCINT4)PB4
- net 8PB5: no longer IC4.(PCINT5)PB5
- net 8PB6: no longer IC4.(PCINT6)PB6
- net 8PB7: no longer IC4.(PCINT7/OC0A/OC1C)PB7
- net ADC0: no longer IC3.(ADC0)PF0
- net ADC1: no longer IC3.(ADC1)PF1
- net ADC10: no longer IC3.PK2(ADC10/PCINT18)
- net ADC11: no longer IC3.PK3(ADC11/PCINT19)
- net ADC12: no longer IC3.PK4(ADC12/PCINT20)
- net ADC13: no longer IC3.PK5(ADC13/PCINT21)
- net ADC14: no longer IC3.PK6(ADC14/PCINT22)
- net ADC15: no longer IC3.PK7(ADC15/PCINT23)
- net ADC2: no longer IC3.(ADC2)PF2
- net ADC3: no longer IC3.(ADC3)PF3
- net ADC4: no longer IC3.(ADC4/TCK)PF4
- net ADC5: no longer IC3.(ADC5/TMS)PF5
- net ADC6: no longer IC3.(ADC6/TDO)PF6
- net ADC7: no longer IC3.(ADC7/TDI)PF7
- net ADC8: no longer IC3.PK0(ADC8/PCINT16)
- net ADC9: no longer IC3.PK1(ADC9/PCINT17)
- net AREF: no longer C3.1, IC3.AREF
- net GND: no longer C1.2, C11.1, C12.1, C13.1, C14.2, C15.2, C2.2, C3.2, C4.2, C5.2, C6.2, C8.2, C9.2, GROUND.2, IC1.GND/ADJ, IC3.AGND, IC3.GND, IC3.GND1, IC3.GND2, IC3.GND3, IC4.GND, IC4.PAD, IC6.GND, IC7P.V-, L.C, ON.C, PC1.-, PC2.-, RESET.1, RESET.2, RN3D.2, RN5D.1, X1.1, X1.3, Y1.2
- net MISO2: no longer IC4.(PD0/MISO/PCINT3)PB3
- net MOSI2: no longer IC4.(PDI/MOSI/PCINT2)PB2
- net N$3: now also JP6.2; no longer ON.A, RN3A.2
- net PA0: no longer IC3.(AD0)PA0
- net PA1: no longer IC3.(AD1)PA1
- net PA2: no longer IC3.(AD2)PA2
- net PA3: no longer IC3.(AD3)PA3
- net PA4: no longer IC3.(AD4)PA4
- net PA5: no longer IC3.(AD5)PA5
- net PA6: no longer IC3.(AD6)PA6
- net PA7: no longer IC3.(AD7)PA7
- net PB0: no longer IC3.(SS/PCINT0)PB0
- net PB1: no longer IC3.(SCK/PCINT1)PB1
- net PB2: no longer IC3.(MOSI/PCINT2)PB2
- net PB3: no longer IC3.(MISO/PCINT3)PB3
- net PB4: no longer IC3.(OC2A/PCINT4)PB4
- net PB5: no longer IC3.(OC1A/PCINT5)PB5
- net PB6: no longer IC3.(OC1B/PCINT6)PB6
- net PB7: no longer IC3.(OC0A/OC1C/PCINT7)PB7, IC7A.+IN
- net PC0: no longer IC3.(A8)PC0
- net PC1: no longer IC3.(A9)PC1
- net PC2: no longer IC3.(A10)PC2
- net PC3: no longer IC3.(A11)PC3
- net PC4: no longer IC3.(A12)PC4
- net PC5: no longer IC3.(A13)PC5
- net PC6: no longer IC3.(A14)PC6
- net PC7: no longer IC3.(A15)PC7
- net PD7: no longer IC3.(T0)PD7
- net PE0: no longer IC3.(RXD0/PCIN8)PE0, RN4B.1
- net PE1: no longer IC3.(TXD0)PE1, RN4A.1
- net PE3: no longer IC3.(OC3A/AIN1)PE3
- net PE4: no longer IC3.(OC3B/INT4)PE4
- net PE5: no longer IC3.(OC3C/INT5)PE5
- net PG0: no longer IC3.(WR)PG0
- net PG1: no longer IC3.(RD)PG1
- net PG2: no longer IC3.(ALE)PG2
- net PG5: no longer IC3.(OC0B)PG5
- net PH3: no longer IC3.PH3(OC4A)
- net PH4: no longer IC3.PH4(OC4B)
- net PH5: no longer IC3.PH5(OC4C)
- net PH6: no longer IC3.PH6(OC2B)
- net PL0: no longer IC3.PL0(ICP4)
- net PL1: no longer IC3.PL1(ICP5)
- net PL2: no longer IC3.PL2(T5)
- net PL3: no longer IC3.PL3(OC5A)
- net PL4: no longer IC3.PL4(OC5B)
- net PL5: no longer IC3.PL5(OC5C)
- net PL6: no longer IC3.PL6
- net PL7: no longer IC3.PL7
- net RESET: now also POWER.1; no longer C1.1, C7.2, D3.A, IC3.RESET, POWER.3, RESET-EN.1, RESET-EN.2, RESET.3, RESET.4, RN5A.1
- net RESET2: no longer D2.A, IC4.RESET(PC1/DW), RN5B.2
- net RXD1: no longer IC3.(RXD1/INT2)PD2
- net RXD2: no longer IC3.PH0(RXD2)
- net RXD3: no longer IC3.PJ0(RXD3/PCINT9)
- net SCK2: no longer IC4.(SCLK/PCINT1)PB1
- net SCL: no longer IC3.(SCL/INT0)PD0, RN1B.1
- net SDA: no longer IC3.(SDA/INT1)PD1, JP6.2, RN1C.1
- net TXD1: no longer IC3.(TXD1/INT3)PD3
- net TXD2: no longer IC3.PH1(TXD2)
- net TXD3: no longer IC3.PJ1(TXD3/PCINT10)
- net VIN: no longer C2.1, D1.C, IC1.IN, PC1.+, RN5C.2
Other:
- note removed: "Arduino MEGA 2560"
- note removed: "TM"
- note removed: "USB boot En"
- moved on the sheet: ADCH, COMMUNICATION, ICSP, ICSP1, JP5, JP6, POWER, PWML, XIO

Commit message: schema work, not final
Parts:
- added CN1: LED-RGB1, adafruit:1X4-BIG
- added CN2: LED-RGB2, adafruit:1X4-BIG
- added CN3: LED-RGB3, adafruit:1X4-BIG
- added JP1: PWM_driver, adafruit:PINHD-1X6
- added JP2, JP4: (no value), adafruit:PINHD-1X8BIG
- added JP3: (no value), microbuilder:HEADER-1X10
- added JP7: (no value), adafruit:PINHD-1X3
- added R1, R2, R3, R4, R5, R6, R7, R8, R9: (no value), adafruit:R-US_0207/10
- JP5: value 2x2M - NM -> (none); device SmartPrj:PINHD-2X2 -> adafruit:PINHD-1X3
Connections:
- removed net 8PB4: JP5.1
- removed net 8PB5: JP5.3
- removed net 8PB6: JP5.2
- removed net 8PB7: JP5.4
- new net N$1: R6.1
- new net N$10: JP2.7
- new net N$11: R4.1
- new net N$12: CN1.3, R5.2
- new net N$15: R3.1
- new net N$2: CN2.3, R2.2
- new net N$20: JP2.5
- new net N$21: R2.1
- new net N$22: R1.1
- new net N$24: JP4.1
- new net N$25: JP4.2
- new net N$29: JP4.6
- new net N$30: JP4.7
- new net N$4: CN3.4, R9.2
- new net N$45: CN3.1, R7.2
- new net N$5: CN1.1, R4.2
- new net N$6: R5.1
- new net N$7: CN3.3, R8.2
- new net N$8: CN1.4, R6.2
- new net N$9: CN2.1, R1.2
- net +5V: now also JP1.2, JP2.6, JP3.1, JP5.2, JP7.2
- net ADC0: now also JP5.1
- net ADC1: now also JP7.1
- net ADC2: now also JP3.10
- net ADC3: now also JP4.8
- net GND: now also CN1.2, CN2.2, CN3.2, JP1.6, JP2.8, JP3.8, JP5.3, JP7.3
- net N$3: now also CN2.4, R3.2; no longer JP6.2
- net PA0: now also JP3.4
- net PA1: now also JP3.5
- net PA2: now also JP3.3
- net PA4: now also JP3.2
- net PA7: now also JP4.3
- net PB2: now also JP2.4
- net PB4: now also R8.1
- net PB5: now also R7.1
- net PC4: now also JP4.4
- net PC6: now also JP4.5
- net PE3: now also JP3.9
- net PE4: now also JP2.3
- net PE5: now also JP2.2
- net PG5: now also JP2.1
- net PH3: now also JP3.7
- net PH4: now also JP3.6
- net PH6: now also R9.1
- net SCL: now also JP1.4
- net SDA: now also JP1.3, JP6.2
Other:
- note added: "???"
- note added: "ENC 1A"
- note added: "ENC 1B"
- note added: "ENC 1SW"
- note added: "ENC1 SW"
- note added: "ENC2 A"
- note added: "ENC2 B"
- note added: "ENC2 SW"
- note added: "KNOB1"
- note added: "KNOB2"
- note added: "LCD BL"
- note added: "LCD CDK"
- note added: "LCD CE"
- note added: "LCD DC"
- note added: "LCD Pin"
- note added: "LCD RST"
- note added: "LED1 B"
- note added: "LED1 G"
- note added: "LED1 R"
- note added: "LED2 B"
- note added: "LED2 G"
- note added: "LED2 R"
- note added: "LED3 B"
- note added: "LED3 G"
- note added: "LED3 R"
- note added: "MUX S0"
- note added: "MUX S1"
- note added: "MUX S2"
- note added: "MUX S3"
- note added: "Mega shield"
- note added: "POT1"
- note added: "POT2"
- moved on the sheet: ADCH, ICSP

Commit message: updates, ready for beutification
Parts:
- removed FD1, FD2, FD3, FD4: FIDUCIALMOUNT, SmartPrj:FIDUCIALMOUNT
- removed ICSP, ICSP1: 3x2M, SmartPrj:PINHD-2X3
- removed JP4: (no value), adafruit:PINHD-1X8BIG
- removed R7, R8, R9: (no value), adafruit:R-US_0207/10
- added CN4: PWM-13/16, adafruit:1X4-BIG
- added JP8: (no value), eduBoard:HEADER-1X5
- added R10: (no value), adafruit:R-US_0207/10
- added S1: (no value), adafruit:EG1218S
- added S2: SWITCH-MOMENTARY-2PTH, eduBoard:SWITCH-MOMENTARY-2PTH
- CN1: value LED-RGB1 -> LED-RGB2
- CN2: value LED-RGB2 -> LED-RGB1
- JP2: device adafruit:PINHD-1X8BIG -> eduBoard:PINHD-1X8OVAL
- JP3: device microbuilder:HEADER-1X10 -> eduBoard:PINHD-1X10_ARD
- renumbered ADCH to ~~~ADC~~~, COMMUNICATION to ~~~COM~~~, POWER to ~~POWER~~, PWML to ~~~PWM~~~
Connections:
- removed net MISO2: ICSP1.1
- removed net MOSI2: ICSP1.4
- removed net N$1: R6.1
- removed net N$11: R4.1
- removed net N$15: R3.1
- removed net N$20: JP2.5
- removed net N$21: R2.1
- removed net N$22: R1.1
- removed net N$24: JP4.1
- removed net N$25: JP4.2
- removed net N$29: JP4.6
- removed net N$30: JP4.7
- removed net N$4: CN3.4, R9.2
- removed net N$45: CN3.1, R7.2
- removed net N$6: R5.1
- removed net N$7: CN3.3, R8.2
- removed net RESET2: ICSP1.5
- removed net SCK2: ICSP1.3
- new net 3V3: JP2.6
- new net IOREF: ~~POWER~~.2
- new net N$13: R10.1, S1.P
- new net PWM13: CN4.1
- new net PWM14: CN3.4, CN4.2
- new net PWM15: CN3.3, CN4.3
- new net PWM16: CN3.1, CN4.4
- net +5V: now also S1.S; no longer ICSP.2, ICSP1.2, JP2.6, ~~POWER~~.2
- net ADC3: now also JP8.2; no longer JP4.8
- net GND: now also S2.1; no longer ICSP.6, ICSP1.6
- net N$10: now also R10.2
- net PA1: now also JP8.1
- net PA7: no longer JP4.3
- net PB1: now also JP2.5; no longer ICSP.3
- net PB2: no longer ICSP.4
- net PB3: no longer ICSP.1
- net PB4: now also R2.1; no longer R8.1
- net PB5: now also R1.1; no longer R7.1
- net PB6: now also R3.1
- net PC4: now also JP8.4; no longer JP4.4
- net PC6: now also JP8.5; no longer JP4.5
- net PC7: now also JP8.3
- net PH6: no longer R9.1
- net PL3: now also R6.1
- net PL4: now also R4.1
- net PL5: now also R5.1
- net RESET: now also S2.2, ~~POWER~~.3; no longer ICSP.5, ~~POWER~~.1
Other:
- note added: "LCD CLK"
- note added: "LCD DIN"
- note added: "MUX sig"
- note removed: "???"
- note removed: "LCD CDK"
- note removed: "LCD Pin"
- moved on the sheet: CN1, CN2, CN3, JP1, R1, R2, R3, R4, R5, R6

Commit message: pushed
Connections:
- removed net 3V3: JP2.6
- net +3V3: now also JP2.6
- net PA1: no longer JP3.5
- net PA6: now also JP3.5

Commit message: routed
Connections:
- net PB4: now also R1.1; no longer R2.1
- net PB5: now also R2.1; no longer R1.1
Changed lines of the file:
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@@
 </segment>
 <segment>
-<pinref part="R1" gate="G$1" pin="1"/>
-<wire x1="7.62" y1="134.62" x2="7.62" y2="124.46" width="0.1524" layer="91"/>
-<label x="7.62" y="124.46" size="1.778" layer="95" rot="R90"/>
+<pinref part="R2" gate="G$1" pin="1"/>
+<wire x1="12.7" y1="132.08" x2="12.7" y2="124.46" width="0.1524" layer="91"/>
+<label x="12.7" y="124.46" size="1.778" layer="95" rot="R90"/>
 </segment>
 </net>
@@
 </segment>
 <segment>
-<pinref part="R2" gate="G$1" pin="1"/>
-<wire x1="12.7" y1="132.08" x2="12.7" y2="124.46" width="0.1524" layer="91"/>
-<label x="12.7" y="124.46" size="1.778" layer="95" rot="R90"/>
+<pinref part="R1" gate="G$1" pin="1"/>
+<wire x1="7.62" y1="134.62" x2="7.62" y2="124.46" width="0.1524" layer="91"/>
+<label x="7.62" y="124.46" size="1.778" layer="95" rot="R90"/>
 </segment>
 </net>
